Commit message: fanuc_description

File: fanuc_description/robot/fanuc.urdf (robot description, URDF)
Before this commit: robot fanuc, 8 links, 7 joints
Links:
- link base_link: geometry collision mesh filename=package://fanuc_description/meshes/collision/link_0.stl; visual mesh filename=package://fanuc_description/meshes/visual/link_0.dae
- link link1: geometry collision mesh filename=package://fanuc_description/meshes/collision/link_1.stl; visual mesh filename=package://fanuc_description/meshes/visual/link_1.dae
- link link2: geometry collision mesh filename=package://fanuc_description/meshes/collision/link_2.stl; visual mesh filename=package://fanuc_description/meshes/visual/link_2.dae
- link link3: geometry collision mesh filename=package://fanuc_description/meshes/collision/link_3.stl; visual mesh filename=package://fanuc_description/meshes/visual/link_3.dae
- link link4: geometry collision mesh filename=package://fanuc_description/meshes/collision/link_4.stl; visual mesh filename=package://fanuc_description/meshes/visual/link_4.dae
- link link5: geometry collision mesh filename=package://fanuc_description/meshes/collision/link_5.stl; visual mesh filename=package://fanuc_description/meshes/visual/link_5.dae
- link link6: geometry collision mesh filename=package://fanuc_description/meshes/collision/link_6.stl; visual mesh filename=package://fanuc_description/meshes/visual/link_6.dae

Commit message: ex2FanucTf

File: fanuc_description/robot/fanuc.urdf (robot description, URDF)
Before this commit: robot fanuc, 8 links, 7 joints
Links:
- added link world
Joints:
- added joint virtual_joint: type fixed, parent world, child base_link
- joint flange: limit lower=-2.967 upper=2.967 effort=12 velocity=2.433 -> (none)
- joint joint1: limit lower=-2.967 upper=2.967 effort=12 velocity=2.433 -> lower=-2.967 upper=2.967 effort=12 velocity=2.443
- joint joint_2: limit lower=-2.967 upper=2.967 effort=12 velocity=2.433 -> lower=-1.4835 upper=2.7052 effort=12 velocity=2.792
- joint joint_3: limit lower=-2.967 upper=2.967 effort=12 velocity=2.433 -> lower=-1.5707 upper=1.3962 effort=12 velocity=2.967
- joint joint_4: limit lower=-2.967 upper=2.967 effort=12 velocity=2.433 -> lower=-3.6651 upper=3.6651 effort=11.7 velocity=10.47
- joint joint_5: limit lower=-2.967 upper=2.967 effort=12 velocity=2.433 -> lower=-2.2689 upper=2.2689 effort=11.7 velocity=6.545
- joint joint_6: limit lower=-2.967 upper=2.967 effort=12 velocity=2.433 -> lower=-47.1238 upper=47.1238 effort=5.8 velocity=9.6
